File: fcu/fcu-kicad-v0.2/fcu-kicad-v0.2.kicad_sch (KiCad schematic)
At the start: 186 parts, among them J1 Conn_01x02, J10 Conn_01x02_Socket, J11 Conn_01x04_Socket, J12 Conn_01x02_Socket, J13 Conn_01x02_Socket, J14 Conn_01x02_Socket, J15 Conn_01x02_Socket, J16 Conn_01x02_Socket, J17 Conn_01x02_Socket, J18 Conn_01x02_Socket, J19 Conn_01x02_Socket, J2 Conn_01x04_Socket, J20 Conn_01x02_Socket, J21 Conn_01x02_Socket, J22 Conn_01x02_Socket, J23 Conn_01x02_Socket, J24 Conn_01x02_Socket, J25 Conn_01x02, J3 Conn_01x01, J4 Conn_01x02_Socket, J5 Conn_01x03_Pin, J6 Conn_01x04_Socket, J7 Conn_01x06_Socket, J8 Conn_01x03_Socket, J9 Conn_01x02_Socket, SW1 SW_RST, U1 MCP1416, U10 RQ3E100, U11 RQ3E100, U12 MS5611-01BA, U13 W25X05, U14 W25X05, U15 LAN8742, U16 MCP1416, U17 MAX-8C, U18 RQ3E100, U19 AP62300TWU, U2 MCP1416, U20 LD39200, U21 TXB0108DQSR, U3 RQ3E100, U4 RQ3E100, U5 STM32F407VGTx, U6 MCP1416, U7 MCP1416, U8 BMM150, U9 BMI088, Y1 25 MHz, Y2 25 MHz

Commit message: Routing work on FCU v0.2
Parts:
- removed C49: 10uF, Capacitor_SMD:C_0402_1005Metric, symbol Device:C_Small
- C38, C43, C46, C48, C50: footprint Capacitor_SMD:C_0402_1005Metric -> Capacitor_SMD:C_0603_1608Metric
Connections:
- net Vdrive: now also J4.2 (Pin_2); no longer J4.1 (Pin_1)
- net at J5.3 (Pin_3), R54.1: now also J4.1 (Pin_1); no longer J4.2 (Pin_2)
Other:
- moved on the sheet: J4
Changed lines of the file:
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@@
   (junction (at 327.66 71.12) (diameter 0) (color 0 0 0 0)
   )
+  (junction (at 492.76 44.45) (diameter 0) (color 0 0 0 0)
+  )
   (junction (at 332.74 276.86) (diameter 0) (color 0 0 0 0)
   )
@@
   (junction (at 86.36 30.48) (diameter 0) (color 0 0 0 0)
   )
-  (junction (at 494.03 35.56) (diameter 0) (color 0 0 0 0)
+  (junction (at 521.97 39.37) (diameter 0) (color 0 0 0 0)
   )
   (junction (at 335.28 73.66) (diameter 0) (color 0 0 0 0)
@@
   (junction (at 118.11 312.42) (diameter 0) (color 0 0 0 0)
   )
-  (junction (at 492.76 44.45) (diameter 0) (color 0 0 0 0)
-  )
   (junction (at 231.14 66.04) (diameter 0) (color 0 0 0 0)
   )
@@
     (stroke (width 0) (type default))
   )
-  (wire (pts (xy 494.03 34.29) (xy 494.03 35.56))
+  (wire (pts (xy 521.97 38.1) (xy 521.97 39.37))
     (stroke (width 0) (type default))
   )
@@
     (stroke (width 0) (type default))
   )
+  (wire (pts (xy 492.76 44.45) (xy 496.57 44.45))
+    (stroke (width 0) (type default))
+  )
+  (wire (pts (xy 495.3 39.37) (xy 495.3 38.1))
+    (stroke (width 0) (type default))
+  )
   (wire (pts (xy 118.11 313.69) (xy 119.38 313.69))
     (stroke (width 0) (type default))
@@
     (stroke (width 0) (type default))
   )
-  (wire (pts (xy 391.16 116.84) (xy 391.16 118.11))
-    (stroke (width 0) (type default))
-  )
   (wire (pts (xy 372.11 72.39) (xy 391.16 72.39))
     (stroke (width 0) (type default))
@@
     (stroke (width 0) (type default))
   )
-  (wire (pts (xy 496.57 38.1) (xy 492.76 38.1))
-    (stroke (width 0) (type default))
-  )
-  (wire (pts (xy 485.14 35.56) (xy 494.03 35.56))
+  (wire (pts (xy 530.86 39.37) (xy 521.97 39.37))
     (stroke (width 0) (type default))
   )
@@
     (stroke (width 0) (type default))
   )
-  (wire (pts (xy 492.76 44.45) (xy 496.57 44.45))
+  (wire (pts (xy 469.9 44.45) (xy 492.76 44.45))
     (stroke (width 0) (type default))
   )
@@
     (stroke (width 0) (type default))
   )
-  (wire (pts (xy 485.14 34.29) (xy 485.14 35.56))
+  (wire (pts (xy 530.86 38.1) (xy 530.86 39.37))
     (stroke (width 0) (type default))
   )
@@
     (stroke (width 0) (type default))
   )
+  (wire (pts (xy 492.76 38.1) (xy 492.76 44.45))
+    (stroke (width 0) (type default))
+  )
   (wire (pts (xy 115.57 118.11) (xy 142.24 118.11))
     (stroke (width 0) (type default))
@@
     (stroke (width 0) (type default))
   )
-  (wire (pts (xy 494.03 35.56) (xy 496.57 35.56))
+  (wire (pts (xy 495.3 39.37) (xy 521.97 39.37))
     (stroke (width 0) (type default))
   )
@@
     (stroke (width 0) (type default))
   )
-  (wire (pts (xy 469.9 44.45) (xy 492.76 44.45))
-    (stroke (width 0) (type default))
-  )
   (wire (pts (xy 124.46 311.15) (xy 125.73 311.15))
     (stroke (width 0) (type default))
@@
     (stroke (width 0) (type default))
   )
-  (wire (pts (xy 492.76 38.1) (xy 492.76 44.45))
-    (stroke (width 0) (type default))
-  )
   (wire (pts (xy 252.73 33.02) (xy 252.73 48.26))
     (stroke (width 0) (type default))
@@
     (effects (font (size 1.27 1.27)) (justify left bottom))
   )
-  (text "Output Arming" (at 508 35.56 0)
+  (text "Output Arming" (at 501.65 33.02 0)
     (effects (font (size 1.27 1.27)) (justify left bottom))
   )
@@
       (effects (font (size 1.27 1.27)) (justify left))
     )
-    (property "Footprint" "Capacitor_SMD:C_0402_1005Metric" (at 339.09 151.13 0)
+    (property "Footprint" "Capacitor_SMD:C_0603_1608Metric" (at 339.09 151.13 0)
       (effects (font (size 1.27 1.27)) hide)
     )
@@
       (effects (font (size 1.27 1.27)) hide)
     )
-    (property "Field5" "" (at 490.22 54.61 0)
-      (effects (font (size 1.27 1.27)) hide)
-    )
     (pin "1")
     (pin "2")
@@
       (effects (font (size 1.27 1.27)) (justify left))
     )
-    (property "Footprint" "Capacitor_SMD:C_0402_1005Metric" (at 381 121.92 0)
+    (property "Footprint" "Capacitor_SMD:C_0603_1608Metric" (at 381 121.92 0)
       (effects (font (size 1.27 1.27)) hide)
     )
@@
     )
   )
-  (symbol (lib_id "power:Vdrive") (at 485.14 34.29 0) (unit 1)
+  (symbol (lib_id "power:Vdrive") (at 530.86 38.1 0) (mirror y) (unit 1)
     (in_bom yes) (on_board yes) (dnp no) (fields_autoplaced)
-    (property "Reference" "#PWR0138" (at 480.06 38.1 0)
+    (property "Reference" "#PWR0138" (at 535.94 41.91 0)
       (effects (font (size 1.27 1.27)) hide)
     )
-    (property "Value" "Vdrive" (at 485.14 30.48 0)
+    (property "Value" "Vdrive" (at 530.86 34.29 0)
       (effects (font (size 1.27 1.27)))
     )
-    (property "Footprint" "" (at 485.14 34.29 0)
+    (property "Footprint" "" (at 530.86 38.1 0)
       (effects (font (size 1.27 1.27)) hide)
     )
-    (property "Datasheet" "" (at 485.14 34.29 0)
+    (property "Datasheet" "" (at 530.86 38.1 0)
       (effects (font (size 1.27 1.27)) hide)
     )
@@
       (effects (font (size 1.27 1.27)) (justify left))
     )
-    (property "Footprint" "Capacitor_SMD:C_0402_1005Metric" (at 320.04 119.38 0)
+    (property "Footprint" "Capacitor_SMD:C_0603_1608Metric" (at 320.04 119.38 0)
       (effects (font (size 1.27 1.27)) hide)
     )
@@
     )
   )
-  (symbol (lib_id "Device:C_Small") (at 391.16 114.3 0) (unit 1)
-    (in_bom yes) (on_board yes) (dnp no) (fields_autoplaced)
-    (property "Reference" "C49" (at 393.7 113.6713 0)
-      (effects (font (size 1.27 1.27)) (justify left))
-    )
-    (property "Value" "10uF" (at 393.7 116.2113 0)
-      (effects (font (size 1.27 1.27)) (justify left))
-    )
-    (property "Footprint" "Capacitor_SMD:C_0402_1005Metric" (at 391.16 114.3 0)
-      (effects (font (size 1.27 1.27)) hide)
-    )
-    (property "Datasheet" "~" (at 391.16 114.3 0)
-      (effects (font (size 1.27 1.27)) hide)
-    )
-    (pin "1")
-    (pin "2")
-    (instances
-      (project "fcu-kicad-v0.2"
-        (path "/29f1fc7e-a327-4eeb-ad25-e83c2280ace8"
-          (reference "C49") (unit 1)
-        )
-      )
-    )
-  )
   (symbol (lib_id "Device:R_Small") (at 247.65 73.66 90) (unit 1)
     (in_bom yes) (on_board yes) (dnp no)
@@
     )
   )
-  (symbol (lib_id "power:GND") (at 391.16 111.76 180) (unit 1)
-    (in_bom yes) (on_board yes) (dnp no) (fields_autoplaced)
-    (property "Reference" "#PWR0123" (at 391.16 105.41 0)
-      (effects (font (size 1.27 1.27)) hide)
-    )
-    (property "Value" "GND" (at 391.16 107.95 0)
-      (effects (font (size 1.27 1.27)))
-    )
-    (property "Footprint" "" (at 391.16 111.76 0)
-      (effects (font (size 1.27 1.27)) hide)
-    )
-    (property "Datasheet" "" (at 391.16 111.76 0)
-      (effects (font (size 1.27 1.27)) hide)
-    )
-    (pin "1")
-    (instances
-      (project "fcu-kicad-v0.2"
-        (path "/29f1fc7e-a327-4eeb-ad25-e83c2280ace8"
-          (reference "#PWR0123") (unit 1)
-        )
-      )
-    )
-  )
   (symbol (lib_id "power:+3.3V") (at 246.38 181.61 270) (unit 1)
     (in_bom yes) (on_board yes) (dnp no)
@@
     )
   )
-  (symbol (lib_id "power:PWR_FLAG") (at 494.03 34.29 0) (unit 1)
+  (symbol (lib_id "power:PWR_FLAG") (at 521.97 38.1 0) (mirror y) (unit 1)
     (in_bom yes) (on_board yes) (dnp no) (fields_autoplaced)
-    (property "Reference" "#FLG05" (at 494.03 32.385 0)
+    (property "Reference" "#FLG05" (at 521.97 36.195 0)
       (effects (font (size 1.27 1.27)) hide)
     )
-    (property "Value" "PWR_FLAG" (at 494.03 30.48 0)
+    (property "Value" "PWR_FLAG" (at 521.97 34.29 0)
       (effects (font (size 1.27 1.27)))
     )
-    (property "Footprint" "" (at 494.03 34.29 0)
+    (property "Footprint" "" (at 521.97 38.1 0)
       (effects (font (size 1.27 1.27)) hide)
     )
-    (property "Datasheet" "~" (at 494.03 34.29 0)
+    (property "Datasheet" "~" (at 521.97 38.1 0)
       (effects (font (size 1.27 1.27)) hide)
     )
@@
       (effects (font (size 1.27 1.27)) (justify left))
     )
-    (property "Footprint" "Capacitor_SMD:C_0402_1005Metric" (at 391.16 121.92 0)
+    (property "Footprint" "Capacitor_SMD:C_0603_1608Metric" (at 391.16 121.92 0)
       (effects (font (size 1.27 1.27)) hide)
     )
@@
       (effects (font (size 1.27 1.27)) (justify left))
     )
-    (property "Footprint" "Capacitor_SMD:C_0402_1005Metric" (at 373.38 153.67 0)
+    (property "Footprint" "Capacitor_SMD:C_0603_1608Metric" (at 373.38 153.67 0)
       (effects (font (size 1.27 1.27)) hide)
     )
@@
     )
   )
-  (symbol (lib_id "Connector:Conn_01x02_Socket") (at 501.65 35.56 0) (unit 1)
+  (symbol (lib_id "Connector:Conn_01x02_Socket") (at 492.76 33.02 90) (unit 1)
     (in_bom yes) (on_board yes) (dnp no) (fields_autoplaced)
-    (property "Reference" "J4" (at 502.92 36.195 0)
-      (effects (font (size 1.27 1.27)) (justify left))
+    (property "Reference" "J4" (at 496.57 33.02 90)
+      (effects (font (size 1.27 1.27)) (justify right))
     )
-    (property "Value" "Conn_01x02_Socket" (at 502.92 38.735 0)
-      (effects (font (size 1.27 1.27)) (justify left))
+    (property "Value" "Conn_01x02_Socket" (at 496.57 35.56 90)
+      (effects (font (size 1.27 1.27)) (justify right))
     )
-    (property "Footprint" "Connector_JST:JST_VH_B2P-VH_1x02_P3.96mm_Vertical" (at 501.65 35.56 0)
+    (property "Footprint" "Connector_JST:JST_VH_B2P-VH_1x02_P3.96mm_Vertical" (at 492.76 33.02 0)
       (effects (font (size 1.27 1.27)) hide)
     )
-    (property "Datasheet" "~" (at 501.65 35.56 0)
+    (property "Datasheet" "~" (at 492.76 33.02 0)
       (effects (font (size 1.27 1.27)) hide)
     )

Commit message: mission-control-ui rocket page + FCU simulation
Parts:
- added JP1: SolderJumper_3_Open, Jumper:SolderJumper-3_P2.0mm_Open_TrianglePad1.0x1.5mm, symbol Jumper:SolderJumper_3_Open
- C19, C20, C34, C6, C7: LCSC (none) -> C52923
- C53: footprint Capacitor_SMD:C_0504_1310Metric -> Capacitor_SMD:C_0603_1608Metric_Pad1.08x0.95mm_HandSolder
- D1, D2, D8, D9: LCSC (none) -> C40542
- D11, D12, D3, D4: LCSC (none) -> C216740
- R1, R14, R15, R16, R17, R34, R39, R4, R5: LCSC (none) -> C25765
- R23, R24, R6, R7: LCSC (none) -> C25756
- R29, R30, R8, R9: LCSC (none) -> C25882
- R52: value 21K -> 10K
- R53: value 2K -> 2.4K
- R54: value 21K -> 20K
- U1, U16, U2, U6, U7: LCSC (none) -> C83775
- U10, U11, U18, U3, U4: LCSC (none) -> C2924212
- U12: footprint Package_LGA:LGA-8_3x5mm_P1.25mm -> CustomFootprints:LGA-8_3x5mm_P1.25mm_HandSolder
- U15: LCSC (none) -> C621425
Connections:
- net +3.3V: now also JP1.3 (B)
- net +5V: now also JP1.1 (A); no longer J7.1 (Pin_1)
- new net: J7.1 (Pin_1), JP1.2 (C)
