File: engine-controller/ecu-kicad-v0.4/pressure.kicad_sch (KiCad schematic)
At the start: 30 parts

Commit message: That's a lot of changes
Parts:
- added C88, C89, C90, C91, C92, C93: 10nF, symbol Device:C_Small
- added R61, R63, R65, R67, R89, R91: 7.5K, symbol Device:R
- added R62, R64, R66, R68, R90, R92: 15K, symbol Device:R
Connections:
- net GND: now also C88.2, C89.2, C90.2, C91.2, C92.2, C93.2, R62.2, R64.2, R66.2, R68.2, R90.2, R92.2
- new net PS10: R61.1
- new net PS11: R63.1
- new net PS12: R65.1
- new net PS13: R67.1
- new net PS14: R89.1
- new net PS15: R91.1
- new net PS_AI10: C88.1, R61.2, R62.1
- new net PS_AI11: C89.1, R63.2, R64.1
- new net PS_AI12: C90.1, R65.2, R66.1
- new net PS_AI13: C91.1, R67.2, R68.1
- new net PS_AI14: C92.1, R89.2, R90.1
- new net PS_AI15: C93.1, R91.2, R92.1
Other:
- moved on the sheet: C78, C79, C80, C81, C82, C83, C84, C85, C86, C87, R69, R70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
