File: engine-controller/ecu-kicad-v0.4/output_drv.kicad_sch (KiCad schematic)
At the start: 8 parts, among them U19 MCP1416, U20 RQ3E100, U23 INA199xxDCK

Commit message: Lots of sim changes oof
Connections:
- net +3.3V is gone; now on net +12V: U23.3 (V+)
Changed lines of the file:
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@@
   (junction (at 103.505 99.06) (diameter 0) (color 0 0 0 0)
   )
+  (junction (at 104.14 71.755) (diameter 0) (color 0 0 0 0)
+  )
   (junction (at 163.195 102.87) (diameter 0) (color 0 0 0 0)
   )
@@
   (junction (at 163.195 97.79) (diameter 0) (color 0 0 0 0)
   )
-  (junction (at 104.14 71.755) (diameter 0) (color 0 0 0 0)
-  )
   (junction (at 170.18 102.87) (diameter 0) (color 0 0 0 0)
   )
@@
     (stroke (width 0) (type default))
   )
-  (wire (pts (xy 98.425 71.755) (xy 104.14 71.755))
-    (stroke (width 0) (type default))
-  )
   (wire (pts (xy 140.335 102.87) (xy 131.445 102.87))
     (stroke (width 0) (type default))
@@
   )
   (wire (pts (xy 119.38 62.865) (xy 121.92 62.865))
+    (stroke (width 0) (type default))
+  )
+  (wire (pts (xy 99.06 71.755) (xy 104.14 71.755))
     (stroke (width 0) (type default))
   )
@@
     (effects (font (size 1.27 1.27)) (justify right))
   )
-  (hierarchical_label "ISENSE" (shape output) (at 98.425 71.755 180) (fields_autoplaced)
+  (hierarchical_label "ISENSE" (shape output) (at 99.06 71.755 180) (fields_autoplaced)
     (effects (font (size 1.27 1.27)) (justify right))
   )
   (hierarchical_label "OUT" (shape input) (at 173.355 102.87 0) (fields_autoplaced)
     (effects (font (size 1.27 1.27)) (justify left))
-  )
-  (symbol (lib_id "power:+3.3V") (at 121.92 79.375 180) (unit 1)
-    (in_bom yes) (on_board yes) (dnp no) (fields_autoplaced)
-    (property "Reference" "#PWR073" (at 121.92 75.565 0)
-      (effects (font (size 1.27 1.27)) hide)
-    )
-    (property "Value" "+3.3V" (at 121.92 83.82 0)
-      (effects (font (size 1.27 1.27)))
-    )
-    (property "Footprint" "" (at 121.92 79.375 0)
-      (effects (font (size 1.27 1.27)) hide)
-    )
-    (property "Datasheet" "" (at 121.92 79.375 0)
-      (effects (font (size 1.27 1.27)) hide)
-    )
-    (pin "1")
-    (instances
-      (project "ecu-kicad-v0.4"
-        (path "/36cc65d2-4dd3-4f51-bcce-4252e60c9ae8/786c8415-1305-4598-963d-843f7f154a96/64f49881-3157-4073-b83e-d9cba26a7f27"
-          (reference "#PWR073") (unit 1)
-        )
-        (path "/36cc65d2-4dd3-4f51-bcce-4252e60c9ae8/786c8415-1305-4598-963d-843f7f154a96/b1d345e9-2e9c-457a-a0b4-7532a447bfe6"
-          (reference "#PWR073") (unit 1)
-        )
-      )
-    )
   )
   (symbol (lib_id "power:GND") (at 100.965 87.63 270) (unit 1)
@@
         )
       )
+    )
+  )
+  (symbol (lib_id "power:+12V") (at 121.92 79.375 180) (unit 1)
+    (in_bom yes) (on_board yes) (dnp no)
+    (property "Reference" "#PWR06" (at 121.92 75.565 0)
+      (effects (font (size 1.27 1.27)) hide)
+    )
+    (property "Value" "+12V" (at 121.92 83.82 0)
+      (effects (font (size 1.27 1.27)))
+    )
+    (property "Footprint" "" (at 121.92 79.375 0)
+      (effects (font (size 1.27 1.27)) hide)
+    )
+    (property "Datasheet" "" (at 121.92 79.375 0)
+      (effects (font (size 1.27 1.27)) hide)
+    )
+    (pin "1")
+    (instances
+      (project "ecu-kicad-v0.4"
+        (path "/36cc65d2-4dd3-4f51-bcce-4252e60c9ae8/786c8415-1305-4598-963d-843f7f154a96/b1d345e9-2e9c-457a-a0b4-7532a447bfe6"
+          (reference "#PWR06") (unit 1)
+        )
+        (path "/36cc65d2-4dd3-4f51-bcce-4252e60c9ae8/786c8415-1305-4598-963d-843f7f154a96/64f49881-3157-4073-b83e-d9cba26a7f27"
+          (reference "#PWR07") (unit 1)
+        )
+      )
