File: engine-controller/ecu-kicad-v0.4/pressure_sense.kicad_sch (KiCad schematic)
At the start: 4 parts

Commit message: Progress on ECU v0.4
Parts:
- C12: footprint (none) -> Capacitor_SMD:C_0402_1005Metric
- R13: footprint (none) -> Resistor_SMD:R_0603_1608Metric; LCSC C25918 -> C23234
- R14: footprint (none) -> Resistor_SMD:R_0402_1005Metric
