File: engine-controller/ecu-kicad-v0.4/pwm_output_drv.kicad_sch (KiCad schematic)
At the start: 3 parts, among them U25 74LVC1G125

Commit message: Progress on ECU v0.4
Parts:
- R51: footprint (none) -> Capacitor_SMD:C_0402_1005Metric
Changed lines of the file:
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@@
       (effects (font (size 1.27 1.27)) hide)
     )
+    (pin "1")
+    (pin "2")
     (pin "3")
     (pin "4")
     (pin "5")
+    (instances
+      (project "ecu-kicad-v0.4"
+        (path "/36cc65d2-4dd3-4f51-bcce-4252e60c9ae8/786c8415-1305-4598-963d-843f7f154a96/c9de32bf-2057-480e-b155-8b8ac5365133"
+          (reference "U25") (unit 1)
+        )
+        (path "/36cc65d2-4dd3-4f51-bcce-4252e60c9ae8/786c8415-1305-4598-963d-843f7f154a96/0d407d98-2492-44f6-9025-ec2321b96b9d"
+          (reference "U8") (unit 1)
+        )
+        (path "/36cc65d2-4dd3-4f51-bcce-4252e60c9ae8/786c8415-1305-4598-963d-843f7f154a96/72014560-c15a-47f6-8117-d6b3fafff65b"
+          (reference "U11") (unit 1)
+        )
+        (path "/36cc65d2-4dd3-4f51-bcce-4252e60c9ae8/786c8415-1305-4598-963d-843f7f154a96/3f75929d-dba2-4d08-a984-5e0c5ba9fe13"
+          (reference "U12") (unit 1)
+        )
+        (path "/36cc65d2-4dd3-4f51-bcce-4252e60c9ae8/786c8415-1305-4598-963d-843f7f154a96/3fe714ca-880f-4160-9f7f-b383c89ee1fe"
+          (reference "U13") (unit 1)
+        )
+        (path "/36cc65d2-4dd3-4f51-bcce-4252e60c9ae8/786c8415-1305-4598-963d-843f7f154a96/bcc73691-ee46-4157-94cc-272d1b60695f"
+          (reference "U14") (unit 1)
+        )
+      )
+    )
+  )
+  (symbol (lib_id "Device:R_Small") (at 96.52 59.055 0) (unit 1)
+    (in_bom yes) (on_board yes) (dnp no)
+    (property "Reference" "R51" (at 97.79 57.785 0)
+      (effects (font (size 1.27 1.27)) (justify left))
+    )
+    (property "Value" "20K" (at 97.79 60.325 0)
+      (effects (font (size 1.27 1.27)) (justify left))
+    )
+    (property "Footprint" "Capacitor_SMD:C_0402_1005Metric" (at 96.52 59.055 0)
+      (effects (font (size 1.27 1.27)) hide)
+    )
+    (property "Datasheet" "~" (at 96.52 59.055 0)
+      (effects (font (size 1.27 1.27)) hide)
+    )
+    (property "LCSC" "C25765" (at 96.52 59.055 0)
+      (effects (font (size 1.27 1.27)) hide)
+    )
     (pin "1")
     (pin "2")
@@
       (project "ecu-kicad-v0.4"
         (path "/36cc65d2-4dd3-4f51-bcce-4252e60c9ae8/786c8415-1305-4598-963d-843f7f154a96/c9de32bf-2057-480e-b155-8b8ac5365133"
-          (reference "U25") (unit 1)
-        )
-      )
-    )
-  )
-  (symbol (lib_id "Device:R_Small") (at 96.52 59.055 0) (unit 1)
-    (in_bom yes) (on_board yes) (dnp no)
-    (property "Reference" "R51" (at 97.79 57.785 0)
-      (effects (font (size 1.27 1.27)) (justify left))
-    )
-    (property "Value" "20K" (at 97.79 60.325 0)
-      (effects (font (size 1.27 1.27)) (justify left))
-    )
-    (property "Footprint" "" (at 96.52 59.055 0)
-      (effects (font (size 1.27 1.27)) hide)
-    )
-    (property "Datasheet" "~" (at 96.52 59.055 0)
-      (effects (font (size 1.27 1.27)) hide)
-    )
-    (property "LCSC" "C25765" (at 96.52 59.055 0)
-      (effects (font (size 1.27 1.27)) hide)
-    )
-    (pin "1")
-    (pin "2")
-    (instances
-      (project "ecu-kicad-v0.4"
-        (path "/36cc65d2-4dd3-4f51-bcce-4252e60c9ae8/786c8415-1305-4598-963d-843f7f154a96/c9de32bf-2057-480e-b155-8b8ac5365133"
           (reference "R51") (unit 1)
+        )
+        (path "/36cc65d2-4dd3-4f51-bcce-4252e60c9ae8/786c8415-1305-4598-963d-843f7f154a96/0d407d98-2492-44f6-9025-ec2321b96b9d"
+          (reference "R10") (unit 1)
+        )
+        (path "/36cc65d2-4dd3-4f51-bcce-4252e60c9ae8/786c8415-1305-4598-963d-843f7f154a96/72014560-c15a-47f6-8117-d6b3fafff65b"
+          (reference "R15") (unit 1)
+        )
+        (path "/36cc65d2-4dd3-4f51-bcce-4252e60c9ae8/786c8415-1305-4598-963d-843f7f154a96/3f75929d-dba2-4d08-a984-5e0c5ba9fe13"
+          (reference "R16") (unit 1)
+        )
+        (path "/36cc65d2-4dd3-4f51-bcce-4252e60c9ae8/786c8415-1305-4598-963d-843f7f154a96/3fe714ca-880f-4160-9f7f-b383c89ee1fe"
+          (reference "R17") (unit 1)
+        )
+        (path "/36cc65d2-4dd3-4f51-bcce-4252e60c9ae8/786c8415-1305-4598-963d-843f7f154a96/bcc73691-ee46-4157-94cc-272d1b60695f"
+          (reference "R18") (unit 1)
         )
       )
@@
           (reference "#PWR085") (unit 1)
         )
+        (path "/36cc65d2-4dd3-4f51-bcce-4252e60c9ae8/786c8415-1305-4598-963d-843f7f154a96/0d407d98-2492-44f6-9025-ec2321b96b9d"
+          (reference "#PWR073") (unit 1)
+        )
+        (path "/36cc65d2-4dd3-4f51-bcce-4252e60c9ae8/786c8415-1305-4598-963d-843f7f154a96/72014560-c15a-47f6-8117-d6b3fafff65b"
+          (reference "#PWR079") (unit 1)
+        )
+        (path "/36cc65d2-4dd3-4f51-bcce-4252e60c9ae8/786c8415-1305-4598-963d-843f7f154a96/3f75929d-dba2-4d08-a984-5e0c5ba9fe13"
+          (reference "#PWR089") (unit 1)
+        )
+        (path "/36cc65d2-4dd3-4f51-bcce-4252e60c9ae8/786c8415-1305-4598-963d-843f7f154a96/3fe714ca-880f-4160-9f7f-b383c89ee1fe"
+          (reference "#PWR093") (unit 1)
+        )
+        (path "/36cc65d2-4dd3-4f51-bcce-4252e60c9ae8/786c8415-1305-4598-963d-843f7f154a96/bcc73691-ee46-4157-94cc-272d1b60695f"
+          (reference "#PWR097") (unit 1)
+        )
       )
     )
@@
         (path "/36cc65d2-4dd3-4f51-bcce-4252e60c9ae8/786c8415-1305-4598-963d-843f7f154a96/c9de32bf-2057-480e-b155-8b8ac5365133"
           (reference "#PWR083") (unit 1)
+        )
+        (path "/36cc65d2-4dd3-4f51-bcce-4252e60c9ae8/786c8415-1305-4598-963d-843f7f154a96/0d407d98-2492-44f6-9025-ec2321b96b9d"
+          (reference "#PWR057") (unit 1)
+        )
+        (path "/36cc65d2-4dd3-4f51-bcce-4252e60c9ae8/786c8415-1305-4598-963d-843f7f154a96/72014560-c15a-47f6-8117-d6b3fafff65b"
+          (reference "#PWR078") (unit 1)
+        )
+        (path "/36cc65d2-4dd3-4f51-bcce-4252e60c9ae8/786c8415-1305-4598-963d-843f7f154a96/3f75929d-dba2-4d08-a984-5e0c5ba9fe13"
+          (reference "#PWR088") (unit 1)
+        )
+        (path "/36cc65d2-4dd3-4f51-bcce-4252e60c9ae8/786c8415-1305-4598-963d-843f7f154a96/3fe714ca-880f-4160-9f7f-b383c89ee1fe"
+          (reference "#PWR092") (unit 1)
+        )
+        (path "/36cc65d2-4dd3-4f51-bcce-4252e60c9ae8/786c8415-1305-4598-963d-843f7f154a96/bcc73691-ee46-4157-94cc-272d1b60695f"
+          (reference "#PWR096") (unit 1)
         )
       )
@@
           (reference "#PWR084") (unit 1)
         )
+        (path "/36cc65d2-4dd3-4f51-bcce-4252e60c9ae8/786c8415-1305-4598-963d-843f7f154a96/0d407d98-2492-44f6-9025-ec2321b96b9d"
+          (reference "#PWR056") (unit 1)
+        )
+        (path "/36cc65d2-4dd3-4f51-bcce-4252e60c9ae8/786c8415-1305-4598-963d-843f7f154a96/72014560-c15a-47f6-8117-d6b3fafff65b"
+          (reference "#PWR075") (unit 1)
+        )
+        (path "/36cc65d2-4dd3-4f51-bcce-4252e60c9ae8/786c8415-1305-4598-963d-843f7f154a96/3f75929d-dba2-4d08-a984-5e0c5ba9fe13"
+          (reference "#PWR087") (unit 1)
+        )
+        (path "/36cc65d2-4dd3-4f51-bcce-4252e60c9ae8/786c8415-1305-4598-963d-843f7f154a96/3fe714ca-880f-4160-9f7f-b383c89ee1fe"
+          (reference "#PWR091") (unit 1)
+        )
+        (path "/36cc65d2-4dd3-4f51-bcce-4252e60c9ae8/786c8415-1305-4598-963d-843f7f154a96/bcc73691-ee46-4157-94cc-272d1b60695f"
+          (reference "#PWR095") (unit 1)
+        )
       )
     )
@@
         (path "/36cc65d2-4dd3-4f51-bcce-4252e60c9ae8/786c8415-1305-4598-963d-843f7f154a96/c9de32bf-2057-480e-b155-8b8ac5365133"
           (reference "C13") (unit 1)
+        )
+        (path "/36cc65d2-4dd3-4f51-bcce-4252e60c9ae8/786c8415-1305-4598-963d-843f7f154a96/0d407d98-2492-44f6-9025-ec2321b96b9d"
+          (reference "C43") (unit 1)
+        )
+        (path "/36cc65d2-4dd3-4f51-bcce-4252e60c9ae8/786c8415-1305-4598-963d-843f7f154a96/72014560-c15a-47f6-8117-d6b3fafff65b"
+          (reference "C44") (unit 1)
+        )
+        (path "/36cc65d2-4dd3-4f51-bcce-4252e60c9ae8/786c8415-1305-4598-963d-843f7f154a96/3f75929d-dba2-4d08-a984-5e0c5ba9fe13"
+          (reference "C51") (unit 1)
+        )
+        (path "/36cc65d2-4dd3-4f51-bcce-4252e60c9ae8/786c8415-1305-4598-963d-843f7f154a96/3fe714ca-880f-4160-9f7f-b383c89ee1fe"
+          (reference "C52") (unit 1)
+        )
+        (path "/36cc65d2-4dd3-4f51-bcce-4252e60c9ae8/786c8415-1305-4598-963d-843f7f154a96/bcc73691-ee46-4157-94cc-272d1b60695f"
+          (reference "C53") (unit 1)
         )
       )
@@
           (reference "#PWR082") (unit 1)
         )
-      )
+        (path "/36cc65d2-4dd3-4f51-bcce-4252e60c9ae8/786c8415-1305-4598-963d-843f7f154a96/0d407d98-2492-44f6-9025-ec2321b96b9d"
+          (reference "#PWR030") (unit 1)
+        )
+        (path "/36cc65d2-4dd3-4f51-bcce-4252e60c9ae8/786c8415-1305-4598-963d-843f7f154a96/72014560-c15a-47f6-8117-d6b3fafff65b"
+          (reference "#PWR074") (unit 1)
+        )
+        (path "/36cc65d2-4dd3-4f51-bcce-4252e60c9ae8/786c8415-1305-4598-963d-843f7f154a96/3f75929d-dba2-4d08-a984-5e0c5ba9fe13"
+          (reference "#PWR086") (unit 1)
+        )
+        (path "/36cc65d2-4dd3-4f51-bcce-4252e60c9ae8/786c8415-1305-4598-963d-843f7f154a96/3fe714ca-880f-4160-9f7f-b383c89ee1fe"
+          (reference "#PWR090") (unit 1)
+        )
+        (path "/36cc65d2-4dd3-4f51-bcce-4252e60c9ae8/786c8415-1305-4598-963d-843f7f154a96/bcc73691-ee46-4157-94cc-272d1b60695f"
+          (reference "#PWR094") (unit 1)
+        )
+      )
