File: engine-controller/ecu-kicad-v0.4/thermocouple_sense.kicad_sch (KiCad schematic)
At the start: 5 parts, among them U1 AD8495

Commit message: Progress on ECU v0.4
Other:
- moved on the sheet: C1, C2, C3, U1
