File: flight-controller/fcu-kicad-v0.2/fcu-kicad-v0.2.kicad_sch (KiCad schematic)
At the start: 186 parts, among them J1 Conn_01x02, J10 Conn_01x02_Socket, J11 Conn_01x04_Socket, J12 Conn_01x02_Socket, J13 Conn_01x02_Socket, J14 Conn_01x02_Socket, J15 Conn_01x02_Socket, J16 Conn_01x02_Socket, J17 Conn_01x02_Socket, J18 Conn_01x02_Socket, J19 Conn_01x02_Socket, J2 Conn_01x04_Socket, J20 Conn_01x02_Socket, J21 Conn_01x02_Socket, J22 Conn_01x02_Socket, J23 Conn_01x02_Socket, J24 Conn_01x02_Socket, J25 Conn_01x02, J3 Conn_01x01, J4 Conn_01x02_Socket, J5 Conn_01x03_Pin, J6 Conn_01x04_Socket, J7 Conn_01x06_Socket, J8 Conn_01x03_Socket, J9 Conn_01x02_Socket, SW1 SW_RST, U1 MCP1416, U10 RQ3E100, U11 RQ3E100, U12 MS5611-01BA, U13 W25X05, U14 W25X05, U15 LAN8742, U16 MCP1416, U17 MAX-8C, U18 RQ3E100, U19 AP62300TWU, U2 MCP1416, U20 LD39200, U21 TXB0108DQSR, U3 RQ3E100, U4 RQ3E100, U5 STM32F407VGTx, U6 MCP1416, U7 MCP1416, U8 BMM150, U9 BMI088, Y1 25 MHz, Y2 25 MHz

Commit message: That's a lot of changes
Parts:
- C8, C9: LCSC (none) -> C12530
Changed lines of the file:
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@@
       (effects (font (size 1.27 1.27)) hide)
     )
+    (property "LCSC" "C12530" (at 66.04 177.8 90)
+      (effects (font (size 1.27 1.27)) hide)
+    )
     (pin "1")
     (pin "2")
@@
       (effects (font (size 1.27 1.27)) hide)
     )
+    (property "LCSC" "C12530" (at 60.96 177.8 90)
+      (effects (font (size 1.27 1.27)) hide)
+    )
